File: TechoSolar.kicad_pcb (KiCad board)
At the start: 2 copper layers, 81.5 x 46.8 mm, 41 parts, among them J1 Conn_02x04_Odd_Even, J2 DE9_Pins, J3 Conn_PIC_ICSP_ICD, J7 Conn_01x02, J8 Conn_01x02, J9 Conn_01x02, SW1 SW_Push, SW2 SW_DIP_x01, SW3 MPB01-1B33-S-D, SW4 MPB01-1B33-S-D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

Commit message: Update TechoSolar.kicad_pcb
Parts:
- moved C16 35.6 mm to (138.0, 75.5)
- moved R3 35.6 mm to (138.0, 78.5)
- moved SW4 28.3 mm to (146.0, 72.0)
- moved U3 18.6 mm to (162.0, 89.0)
- moved R7 17.2 mm to (168.5, 89.0)
- moved J3 17.1 mm to (159.0, 83.5), turned to 90 degrees
Routing:
- net CANRX: track 32.3 -> 8.35 mm, vias 4 -> 2
- net CANTX: track 29.2 -> 8.49 mm
- net GND: track 74.1 -> 53.9 mm, vias 172 -> 165
- net +3.3V: track 154.8 -> 172.7 mm, vias 8 -> 9
- net PGD: track 20.6 -> 13.3 mm, vias 2 -> 1
- net SWI2: track 25.7 -> 33.0 mm, vias 2 -> 1
- net CANL: track 29.5 -> 35.5 mm, vias 0 -> 1
- net PGC: track 21.7 -> 16.1 mm, vias 2 -> 1
- net CANH: track 39.0 -> 42.3 mm
- net MCLR: track 56.7 -> 58.3 mm, vias 3 -> 2
- net SWI1: track 21.7 -> 22.3 mm
- removed copper zone on F.Cu, net +3.3V

Commit message: Update TechoSolar.kicad_pcb
Parts:
- added G***: LOGO, User_Library:logoUB, F.Cu at (111.5, 99.0)
Other:
- board text added: "10/04/2025"
- board text added: "EDD 2025 Miguelangel M. Marc B."
- board text added: "v2. 10/04"
