File: TechoSolar.kicad_sch (KiCad schematic)
At the start: 44 parts, among them J1 Conn_02x04_Odd_Even, J2 DE9_Pins, J3 Conn_PIC_ICSP_ICD, J7 Conn_01x02, J8 Conn_01x02, J9 Conn_01x02, SW1 SW_Push, SW2 SW_Push, SW3 MPB01-1B33-S-D, SW4 MPB01-1B33-S-D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

Commit message: Update TechoSolar.kicad_sch
Parts:
- removed R13, R14: 10k, Resistor_SMD:R_0805_2012Metric_Pad1.20x1.40mm_HandSolder, symbol Device:R
- removed SW2: SW_Push, User_Library:SS01GPD, symbol Switch:SW_Push
- removed U4: LM358, symbol Amplifier_Operational:LM358
- removed U5: LT1117-3.3, symbol Regulator_Linear:LT1117-3.3
- added SW2: SW_DIP_x01, Button_Switch_THT:SW_DIP_SPSTx01_Slide_6.7x4.1mm_W7.62mm_P2.54mm_LowProfile, symbol Switch:SW_DIP_x01
- added U4: LT1117CST-3.3, User_Library:REG_LT1117CST-3.3, symbol LT1117CST-3.3:LT1117CST-3.3
- D1: footprint LED_SMD:LED_0201_0603Metric -> LED_SMD:LED_0603_1608Metric
- J3: footprint (none) -> Connector_PinSocket_2.54mm:PinSocket_1x06_P2.54mm_Vertical
Connections:
- net +12V: now also U4.3 (IN)
- net +3.3V: now also SW2.2, U4.2 (OUT), U4.4 (OUT); no longer J2.9
- net COM: now also SW2.1
- net ENABLE: now also U1.12 (RC4/SDI/SDA); no longer U1.23 (RB5/KBI1/PGM)
- net GND: now also U1.29 (EXP), U4.1 (ADJ/GND); no longer J2.3, J2.6
- net ADC1: no longer names the net of U1.18 (RB0/INT0/AN10)
- net ADC2: no longer names the net of U1.19 (RB1/INT1/AN8)
- net SENSE_1: no longer names the net of U1.3 (RA4/T0CKI)
- net SENSE_2: no longer names the net of U1.4 (RA5/AN4/~{SS}/HLVDIN)
- no-connect marks 13 -> 19
Other:
- note removed: "ADC"
- moved on the sheet: C3, C4

Commit message: Update TechoSolar.kicad_sch
Parts:
- removed C13: 100nF, Capacitor_SMD:C_0603_1608Metric_Pad1.08x0.95mm_HandSolder, symbol Device:C
Other:
- moved on the sheet: C1, C17, C19, C2, C20, C3, C4, J2, J3, R10, R12, R7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

Commit message: Update TechoSolar.kicad_sch
Parts:
- U3: footprint User_Library:SOIC127P599X175-8N -> Package_SO:SOIC-8_3.9x4.9mm_P1.27mm
Changed lines of the file:
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@@
 			)
 		)
-		(property "Footprint" "User_Library:SOIC127P599X175-8N"
+		(property "Footprint" "Package_SO:SOIC-8_3.9x4.9mm_P1.27mm"
 			(at 228.6 44.45 0)
 			(effects

Commit message: Update TechoSolar.kicad_sch
Parts:
- U3: footprint Package_SO:SOIC-8_3.9x4.9mm_P1.27mm -> User_Library:SOIC127P599X175-8N
Changed lines of the file:
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@@
 			)
 		)
-		(property "Footprint" "Package_SO:SOIC-8_3.9x4.9mm_P1.27mm"
+		(property "Footprint" "User_Library:SOIC127P599X175-8N"
 			(at 228.6 44.45 0)
 			(effects

Commit message: Update TechoSolar.kicad_sch
Other:
- note added: "V2_03/04"
- note removed: "V1_2703"
Changed lines of the file:
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@@
 	(generator_version "9.0")
 	(paper "A4")
-	(text "V1_2703"
+	(text "V2_03/04"
 		(exclude_from_sim no)
 		(at 267.462 181.102 0)
